File: Schematics_H-Bridge/ATM_Driver.sch (KiCad schematic (older format))
At the start: 13 parts, among them IC1 ATMEGA328-P, P4 CONN_02X03, SW1 SW_PUSH, U27 7805, Y1 Crystal

Commit message: routing of H-bridge traces
Parts:
- removed IC1: ATMEGA328-P, Housings_DIP:DIP-28_W7.62mm_LongPads, symbol ATMEGA328-P
- removed SW1: SW_PUSH, Buttons_Switches_ThroughHole:KSA_Tactile_SPST, symbol SW_PUSH
- removed U27: 7805, TO_SOT_Packages_THT:TO-220_Neutral123_Vertical_LargePads, symbol 7805
- added SW1: SW_Push, Buttons_Switches_THT:SW_PUSH_6mm, symbol SW_Push
- added U27: L7805, TO_SOT_Packages_THT:TO-220_Horizontal, symbol L7805
- added U28: ATMEGA328P-PU, Housings_DIP:DIP-28_W7.62mm_Socket_LongPads, symbol ATMEGA328P-PU
- C3, C5, C6, C7, C8: footprint Capacitors_ThroughHole:C_Disc_D3_P2.5 -> Capacitors_THT:C_Disc_D4.7mm_W2.5mm_P5.00mm
- C4: footprint Capacitors_ThroughHole:C_Disc_D3_P2.5 -> Capacitors_THT:CP_Radial_D6.3mm_P2.50mm
- R6: footprint Resistors_ThroughHole:Resistor_Horizontal_RM7mm -> Resistors_THT:R_Axial_DIN0204_L3.6mm_D1.6mm_P5.08mm_Horizontal
- R7: footprint Buttons_Switches_ThroughHole:KSA_Tactile_SPST -> Resistors_THT:R_Axial_DIN0204_L3.6mm_D1.6mm_P5.08mm_Horizontal
- Y1: footprint Crystals:HC-49V -> Crystals:Crystal_HC49-4H_Vertical
Connections:
- wire segments 57 -> 58
Other:
- moved on the sheet: C5
Changed lines of the file:
@@
 LIBS:valves
 LIBS:FlipDotComponents
+LIBS:switches
+LIBS:Flipdot_H-Bridge-cache
 EELAYER 25 0
 EELAYER END
@@
 $EndDescr
 $Comp
-L ATMEGA328-P IC1
-U 1 1 58520868
-P 5350 3500
-F 0 "IC1" H 4600 4750 50  0000 L BNN
-F 1 "ATMEGA328-P" H 5750 2100 50  0000 L BNN
-F 2 "Housings_DIP:DIP-28_W7.62mm_LongPads" H 5350 3500 50  0001 C CIN
-F 3 "" H 5350 3500 50  0000 C CNN
-	1    5350 3500
-	1    0    0    -1
-$EndComp
-$Comp
-L 7805 U27
-U 1 1 58520A02
-P 2800 2000
-F 0 "U27" H 2950 1804 50  0000 C CNN
-F 1 "7805" H 2800 2200 50  0000 C CNN
-F 2 "TO_SOT_Packages_THT:TO-220_Neutral123_Vertical_LargePads" H 2800 2000 50  0001 C CNN
-F 3 "" H 2800 2000 50  0000 C CNN
-	1    2800 2000
-	1    0    0    -1
-$EndComp
-$Comp
 L +12V #PWR094
 U 1 1 58520AAA
@@
 F 0 "C3" H 2325 2300 50  0000 L CNN
 F 1 "0.33uF" H 2325 2100 50  0000 L CNN
-F 2 "Capacitors_ThroughHole:C_Disc_D3_P2.5" H 2338 2050 50  0001 C CNN
+F 2 "Capacitors_THT:C_Disc_D4.7mm_W2.5mm_P5.00mm" H 2338 2050 50  0001 C CNN
 F 3 "" H 2300 2200 50  0000 C CNN
 	1    2300 2200
@@
 F 0 "C4" H 3275 2300 50  0000 L CNN
 F 1 "1uF" H 3275 2100 50  0000 L CNN
-F 2 "Capacitors_ThroughHole:C_Disc_D3_P2.5" H 3288 2050 50  0001 C CNN
+F 2 "Capacitors_THT:CP_Radial_D6.3mm_P2.50mm" H 3288 2050 50  0001 C CNN
 F 3 "" H 3250 2200 50  0000 C CNN
 	1    3250 2200
@@
 F 0 "Y1" H 7800 3300 50  0000 C CNN
 F 1 "Crystal" H 7800 3000 50  0000 C CNN
-F 2 "Crystals:HC-49V" H 7800 3150 50  0001 C CNN
+F 2 "Crystals:Crystal_HC49-4H_Vertical" H 7800 3150 50  0001 C CNN
 F 3 "" H 7800 3150 50  0000 C CNN
 	1    7800 3150
@@
 F 0 "R6" V 6880 3850 50  0000 C CNN
 F 1 "10k" V 6800 3850 50  0000 C CNN
-F 2 "Resistors_ThroughHole:Resistor_Horizontal_RM7mm" V 6730 3850 50  0001 C CNN
+F 2 "Resistors_THT:R_Axial_DIN0204_L3.6mm_D1.6mm_P5.08mm_Horizontal" V 6730 3850 50  0001 C CNN
 F 3 "" H 6800 3850 50  0000 C CNN
 	1    6800 3850
 	0    1    1    0
-$EndComp
-$Comp
-L SW_PUSH SW1
-U 1 1 5852197D
-P 7550 3550
-F 0 "SW1" H 7700 3660 50  0000 C CNN
-F 1 "SW_PUSH" H 7550 3470 50  0000 C CNN
-F 2 "Buttons_Switches_ThroughHole:KSA_Tactile_SPST" H 7550 3550 50  0001 C CNN
-F 3 "" H 7550 3550 50  0000 C CNN
-	1    7550 3550
-	1    0    0    -1
 $EndComp
 Text HLabel 6350 4000 2    60   Input ~ 0
@@
 F 0 "C6" H 8175 3100 50  0000 L CNN
 F 1 "22p" H 8175 2900 50  0000 L CNN
-F 2 "Capacitors_ThroughHole:C_Disc_D3_P2.5" H 8188 2850 50  0001 C CNN
+F 2 "Capacitors_THT:C_Disc_D4.7mm_W2.5mm_P5.00mm" H 8188 2850 50  0001 C CNN
 F 3 "" H 8150 3000 50  0000 C CNN
 	1    8150 3000
@@
 F 0 "C7" H 8175 3400 50  0000 L CNN
 F 1 "22p" H 8175 3200 50  0000 L CNN
-F 2 "Capacitors_ThroughHole:C_Disc_D3_P2.5" H 8188 3150 50  0001 C CNN
+F 2 "Capacitors_THT:C_Disc_D4.7mm_W2.5mm_P5.00mm" H 8188 3150 50  0001 C CNN
 F 3 "" H 8150 3300 50  0000 C CNN
 	1    8150 3300
@@
 F 0 "R7" V 7480 3150 50  0000 C CNN
 F 1 "1M" V 7400 3150 50  0000 C CNN
-F 2 "Buttons_Switches_ThroughHole:KSA_Tactile_SPST" V 7330 3150 50  0001 C CNN
+F 2 "Resistors_THT:R_Axial_DIN0204_L3.6mm_D1.6mm_P5.08mm_Horizontal" V 7330 3150 50  0001 C CNN
 F 3 "" H 7400 3150 50  0000 C CNN
 	1    7400 3150
@@
 L C C5
 U 1 1 5997471F
-P 3750 2600
-F 0 "C5" H 3775 2700 50  0000 L CNN
-F 1 "100nF" H 3775 2500 50  0000 L CNN
-F 2 "Capacitors_ThroughHole:C_Disc_D3_P2.5" H 3788 2450 50  0001 C CNN
-F 3 "" H 3750 2600 50  0000 C CNN
-	1    3750 2600
+P 3750 2700
+F 0 "C5" H 3775 2800 50  0000 L CNN
+F 1 "100nF" H 3775 2600 50  0000 L CNN
+F 2 "Capacitors_THT:C_Disc_D4.7mm_W2.5mm_P5.00mm" H 3788 2550 50  0001 C CNN
+F 3 "" H 3750 2700 50  0000 C CNN
+	1    3750 2700
 	1    0    0    -1
 $EndComp
@@
 	2150 1700 2150 1950
 Wire Wire Line
-	2150 1950 2400 1950
-Wire Wire Line
-	3200 1950 8350 1950
+	2150 1950 2500 1950
+Wire Wire Line
+	3100 1950 8350 1950
 Wire Wire Line
 	3750 2400 4450 2400
@@
 	6500 3550 7250 3550
 Wire Wire Line
-	7850 3550 8350 3550
+	7650 3550 8350 3550
 Connection ~ 8350 3550
 Wire Wire Line
@@
 Connection ~ 7400 3300
 Wire Wire Line
-	3750 2400 3750 2450
-Wire Wire Line
-	3750 2750 3750 4600
+	3750 2400 3750 2550
+Wire Wire Line
+	3750 2850 3750 4600
 Connection ~ 3750 4600
 $Comp
@@
 F 0 "C8" H 4125 3350 50  0000 L CNN
 F 1 "100nF" H 4125 3150 50  0000 L CNN
-F 2 "Capacitors_ThroughHole:C_Disc_D3_P2.5" H 4138 3100 50  0001 C CNN
+F 2 "Capacitors_THT:C_Disc_D4.7mm_W2.5mm_P5.00mm" H 4138 3100 50  0001 C CNN
 F 3 "" H 4100 3250 50  0000 C CNN
 	1    4100 3250
 	1    0    0    -1
 $EndComp
-Wire Wire Line
-	4100 3000 4100 3100
 Wire Wire Line
 	4100 3400 4100 3500
@@
 	1    0    0    -1
 $EndComp
+$Comp
+L ATMEGA328P-PU U28
+U 1 1 59AC31FE
+P 5350 3500
+F 0 "U28" H 4600 4750 50  0000 L BNN
+F 1 "ATMEGA328P-PU" H 5750 2100 50  0000 L BNN
+F 2 "Housings_DIP:DIP-28_W7.62mm_Socket_LongPads" H 5350 3500 50  0001 C CIN
+F 3 "" H 5350 3500 50  0001 C CNN
+	1    5350 3500
+	1    0    0    -1
+$EndComp
+$Comp
+L SW_Push SW1
+U 1 1 59AC3D13
+P 7450 3550
+F 0 "SW1" H 7500 3650 50  0000 L CNN
+F 1 "SW_Push" H 7450 3490 50  0000 C CNN
+F 2 "Buttons_Switches_THT:SW_PUSH_6mm" H 7450 3750 50  0001 C CNN
+F 3 "" H 7450 3750 50  0001 C CNN
+	1    7450 3550
+	1    0    0    -1
+$EndComp
+$Comp
+L L7805 U27
+U 1 1 59AC59A7
+P 2800 1950
+F 0 "U27" H 2650 2075 50  0000 C CNN
+F 1 "L7805" H 2800 2075 50  0000 L CNN
+F 2 "TO_SOT_Packages_THT:TO-220_Horizontal" H 2825 1800 50  0001 L CIN
+F 3 "" H 2800 1900 50  0001 C CNN
+	1    2800 1950
+	1    0    0    -1
+$EndComp
+Connection ~ 4100 1950
+Wire Wire Line
+	4100 3000 4100 3100
+Wire Wire Line
+	4100 1950 4100 2700
 $EndSCHEMATC
