File: Schematics_H-Bridge/ATM_Driver.sch (KiCad schematic (older format))
At the start: 13 parts, among them P4 CONN_02X03, SW1 SW_Push, U27 L7805, U28 ATMEGA328P-PU, Y1 Crystal

Commit message: gernerated Gerber and drill files in plot/
Parts:
- R6, R7: footprint Resistors_THT:R_Axial_DIN0204_L3.6mm_D1.6mm_P5.08mm_Horizontal -> Resistors_THT:R_Axial_DIN0204_L3.6mm_D1.6mm_P2.54mm_Vertical
- U27: footprint TO_SOT_Packages_THT:TO-220_Horizontal -> TO_SOT_Packages_THT:TO-220_Vertical
Changed lines of the file:
@@
 F 0 "R6" V 6880 3850 50  0000 C CNN
 F 1 "10k" V 6800 3850 50  0000 C CNN
-F 2 "Resistors_THT:R_Axial_DIN0204_L3.6mm_D1.6mm_P5.08mm_Horizontal" V 6730 3850 50  0001 C CNN
+F 2 "Resistors_THT:R_Axial_DIN0204_L3.6mm_D1.6mm_P2.54mm_Vertical" V 6730 3850 50  0001 C CNN
 F 3 "" H 6800 3850 50  0000 C CNN
 	1    6800 3850
@@
 F 0 "R7" V 7480 3150 50  0000 C CNN
 F 1 "1M" V 7400 3150 50  0000 C CNN
-F 2 "Resistors_THT:R_Axial_DIN0204_L3.6mm_D1.6mm_P5.08mm_Horizontal" V 7330 3150 50  0001 C CNN
+F 2 "Resistors_THT:R_Axial_DIN0204_L3.6mm_D1.6mm_P2.54mm_Vertical" V 7330 3150 50  0001 C CNN
 F 3 "" H 7400 3150 50  0000 C CNN
 	1    7400 3150
@@
 F 0 "U27" H 2650 2075 50  0000 C CNN
 F 1 "L7805" H 2800 2075 50  0000 L CNN
-F 2 "TO_SOT_Packages_THT:TO-220_Horizontal" H 2825 1800 50  0001 L CIN
+F 2 "TO_SOT_Packages_THT:TO-220_Vertical" H 2825 1800 50  0001 L CIN
 F 3 "" H 2800 1900 50  0001 C CNN
 	1    2800 1950
