File: Schematics_H-Bridge/Flipdot_H-Bridge.sch (KiCad schematic (older format))
At the start: 40 parts, among them CON1 BARREL_JACK, P1 CONN_02X13, P2 CONN_02X08, P3 CONN_02X08, U1 74HC595, U10 L293D, U11 L293D, U12 L293D, U13 74HC595, U14 L293D, U15 L293D, U16 L293D, U17 L293D, U18 L293D, U19 L293D, U2 74HC595, U20 ESP8266_D1_Mini, U21 L293D, U22 L293D, U23 L293D, U24 L293D, U25 L293D, U26 L293D, U3 L293D, U4 L293D, U5 L293D, U6 L293D, U7 74HC595, U8 74HC595, U9 L293D

Commit message: routing of H-bridge traces
Parts:
- removed CON1: BARREL_JACK, Connect:BARREL_JACK, symbol BARREL_JACK-RESCUE-Flipdot_H-Bridge
- added J1: Barrel_Jack, Connectors:BARREL_JACK, symbol Barrel_Jack-RESCUE-Flipdot_H-Bridge
- C1: footprint Capacitors_ThroughHole:C_Disc_D3_P2.5 -> Capacitors_THT:C_Disc_D4.7mm_W2.5mm_P5.00mm
- C2: footprint Capacitors_ThroughHole:C_Disc_D6_P5 -> Capacitors_THT:CP_Radial_D6.3mm_P2.50mm
- D1, D2, D3: footprint LEDs:LED-3MM -> LEDs:LED_D3.0mm
- R1, R2, R3, R4, R5: footprint Resistors_ThroughHole:Resistor_Horizontal_RM7mm -> Resistors_THT:R_Axial_DIN0204_L3.6mm_D1.6mm_P5.08mm_Horizontal
- U1, U10, U11, U12, U13, U14, U15, U16, U17, U18, U19, U2, U21, U22, U23, U24, U25, U26, U3, U4, U5, U6, U7, U8, U9: footprint Housings_DIP:DIP-16_W7.62mm_LongPads -> Housings_DIP:DIP-16_W7.62mm_Socket_LongPads
Connections:
- wire segments 546 -> 545
