File: Schematics_H-Bridge/Flipdot_H-Bridge.sch (KiCad schematic (older format))
At the start: 40 parts, among them J1 Barrel_Jack, P1 CONN_02X13, P2 CONN_02X08, P3 CONN_02X08, U1 74HC595, U10 L293D, U11 L293D, U12 L293D, U13 74HC595, U14 L293D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

Commit message: gernerated Gerber and drill files in plot/
Parts:
- R1, R2, R3, R4, R5: footprint Resistors_THT:R_Axial_DIN0204_L3.6mm_D1.6mm_P5.08mm_Horizontal -> Resistors_THT:R_Axial_DIN0204_L3.6mm_D1.6mm_P2.54mm_Vertical
Changed lines of the file:
@@
 F 0 "R1" V 8830 2500 50  0000 C CNN
 F 1 "1k" V 8750 2500 50  0000 C CNN
-F 2 "Resistors_THT:R_Axial_DIN0204_L3.6mm_D1.6mm_P5.08mm_Horizontal" V 8680 2500 50  0001 C CNN
+F 2 "Resistors_THT:R_Axial_DIN0204_L3.6mm_D1.6mm_P2.54mm_Vertical" V 8680 2500 50  0001 C CNN
 F 3 "" H 8750 2500 50  0000 C CNN
 	1    8750 2500
@@
 F 0 "R2" V 8830 3000 50  0000 C CNN
 F 1 "2k" V 8750 3000 50  0000 C CNN
-F 2 "Resistors_THT:R_Axial_DIN0204_L3.6mm_D1.6mm_P5.08mm_Horizontal" V 8680 3000 50  0001 C CNN
+F 2 "Resistors_THT:R_Axial_DIN0204_L3.6mm_D1.6mm_P2.54mm_Vertical" V 8680 3000 50  0001 C CNN
 F 3 "" H 8750 3000 50  0000 C CNN
 	1    8750 3000
@@
 F 0 "R3" V 8380 1900 50  0000 C CNN
 F 1 "1.5K" V 8300 1900 50  0000 C CNN
-F 2 "Resistors_THT:R_Axial_DIN0204_L3.6mm_D1.6mm_P5.08mm_Horizontal" V 8230 1900 50  0001 C CNN
+F 2 "Resistors_THT:R_Axial_DIN0204_L3.6mm_D1.6mm_P2.54mm_Vertical" V 8230 1900 50  0001 C CNN
 F 3 "" H 8300 1900 50  0000 C CNN
 	1    8300 1900
@@
 F 0 "R4" V 8530 1900 50  0000 C CNN
 F 1 "1.5K" V 8450 1900 50  0000 C CNN
-F 2 "Resistors_THT:R_Axial_DIN0204_L3.6mm_D1.6mm_P5.08mm_Horizontal" V 8380 1900 50  0001 C CNN
+F 2 "Resistors_THT:R_Axial_DIN0204_L3.6mm_D1.6mm_P2.54mm_Vertical" V 8380 1900 50  0001 C CNN
 F 3 "" H 8450 1900 50  0000 C CNN
 	1    8450 1900
@@
 F 0 "R5" V 8680 1900 50  0000 C CNN
 F 1 "1.5K" V 8600 1900 50  0000 C CNN
-F 2 "Resistors_THT:R_Axial_DIN0204_L3.6mm_D1.6mm_P5.08mm_Horizontal" V 8530 1900 50  0001 C CNN
+F 2 "Resistors_THT:R_Axial_DIN0204_L3.6mm_D1.6mm_P2.54mm_Vertical" V 8530 1900 50  0001 C CNN
 F 3 "" H 8600 1900 50  0000 C CNN
 	1    8600 1900

Commit message: updated schematic plots plots
Other:
- moved on the sheet: C1, D1, D2, D3, R1, R2, R3, R4, R5, U20

Commit message: PCB v1.1, minor fixes in connector and silkscreen layout
Parts:
- P1: symbol CONN_02X13 -> Conn_02x12_Odd_Even
Connections:
- no-connect marks 37 -> 35
Changed lines of the file:
@@
 $EndComp
 $Comp
-L CONN_02X13 P1
+L Conn_02x12_Odd_Even P1
 U 1 1 58504C7F
-P 13300 3550
-F 0 "P1" H 13300 4250 50  0000 C CNN
-F 1 "CONN_02X13" V 13300 3550 50  0000 C CNN
-F 2 "Pin_Headers:Pin_Header_Straight_2x13_Pitch2.54mm" H 13300 2400 50  0001 C CNN
-F 3 "" H 13300 2400 50  0000 C CNN
-	1    13300 3550
+P 13250 3450
+F 0 "P1" H 13250 4150 50  0000 C CNN
+F 1 "CONN_02X13" V 13250 3450 50  0000 C CNN
+F 2 "Pin_Headers:Pin_Header_Straight_2x13_Pitch2.54mm" H 13250 2300 50  0001 C CNN
+F 3 "" H 13250 2300 50  0000 C CNN
+	1    13250 3450
 	1    0    0    -1
 $EndComp
@@
 Wire Wire Line
 	13700 4050 13550 4050
-NoConn ~ 13050 4150
-NoConn ~ 13550 4150
 Text Label 1550 5150 2    60   ~ 0
 X1

Commit message: removed old ESP code
Parts:
- P1: symbol Conn_02x12_Odd_Even -> CONN_02X13
Connections:
- no-connect marks 35 -> 37
Changed lines of the file:
@@
 $EndComp
 $Comp
-L Conn_02x12_Odd_Even P1
+L CONN_02X13 P1
 U 1 1 58504C7F
-P 13250 3450
-F 0 "P1" H 13250 4150 50  0000 C CNN
-F 1 "CONN_02X13" V 13250 3450 50  0000 C CNN
-F 2 "Pin_Headers:Pin_Header_Straight_2x13_Pitch2.54mm" H 13250 2300 50  0001 C CNN
-F 3 "" H 13250 2300 50  0000 C CNN
-	1    13250 3450
+P 13300 3550
+F 0 "P1" H 13300 4250 50  0000 C CNN
+F 1 "CONN_02X13" V 13300 3550 50  0000 C CNN
+F 2 "Pin_Headers:Pin_Header_Straight_2x13_Pitch2.54mm" H 13300 2400 50  0001 C CNN
+F 3 "" H 13300 2400 50  0000 C CNN
+	1    13300 3550
 	1    0    0    -1
 $EndComp
@@
 Wire Wire Line
 	13700 4050 13550 4050
+NoConn ~ 13050 4150
+NoConn ~ 13550 4150
 Text Label 1550 5150 2    60   ~ 0
 X1
