File: Schematics_H-Bridge/Flipdot_H-Bridge.kicad_pcb (KiCad board)
At the start: 2 copper layers, 53 parts, among them J1 Barrel_Jack, P1 CONN_02X13, P2 CONN_02X08, P3 CONN_02X08, P4 CONN_02X03, SW1 SW_Push, U1 74HC595, U10 L293D, U11 L293D, U12 L293D, U13 74HC595, U14 L293D, U15 L293D, U16 L293D, U17 L293D, U18 L293D, U19 L293D, U2 74HC595, U20 ESP8266_D1_Mini, U21 L293D, U22 L293D, U23 L293D, U24 L293D, U25 L293D, U26 L293D, U27 L7805, U28 ATMEGA328P-PU, U3 L293D, U4 L293D, U5 L293D, U6 L293D, U7 74HC595, U8 74HC595, U9 L293D, Y1 Crystal

Commit message: finished layout V1
Parts:
- added G***: LOGO, FDD_footprint:FDD_Icon, B.Cu at (101.7, 82.3)
- added REF**: VIA-0.6mm, FDD_footprint:VIA-0.6mm, F.Cu at (84.0, 30.5)
- added REF**: VIA-0.6mm, FDD_footprint:VIA-0.6mm, F.Cu at (81.0, 27.5)
- added REF**: VIA-0.6mm, FDD_footprint:VIA-0.6mm, F.Cu at (84.0, 26.5)
- added REF**: VIA-0.6mm, FDD_footprint:VIA-0.6mm, F.Cu at (82.0, 26.5)
- added REF**: VIA-0.6mm, FDD_footprint:VIA-0.6mm, F.Cu at (80.0, 26.5)
- added REF**: VIA-0.6mm, FDD_footprint:VIA-0.6mm, F.Cu at (43.2, 69.7)
- added REF**: VIA-0.6mm, FDD_footprint:VIA-0.6mm, F.Cu at (34.4, 69.7)
- added REF**: VIA-0.6mm, FDD_footprint:VIA-0.6mm, F.Cu at (48.8, 82.8)
- added REF**: VIA-0.6mm, FDD_footprint:VIA-0.6mm, F.Cu at (48.8, 79.4)
- added REF**: VIA-0.6mm, FDD_footprint:VIA-0.6mm, F.Cu at (71.9, 113.5)
- added REF**: VIA-0.6mm, FDD_footprint:VIA-0.6mm, F.Cu at (122.8, 96.4)
- added REF**: VIA-0.6mm, FDD_footprint:VIA-0.6mm, F.Cu at (82.0, 30.5)
- added REF**: VIA-0.6mm, FDD_footprint:VIA-0.6mm, F.Cu at (105.4, 97.9)
- added REF**: VIA-0.6mm, FDD_footprint:VIA-0.6mm, F.Cu at (105.4, 99.6)
- added REF**: MountingHole_5.3mm_M5_DIN965, Mounting_Holes:MountingHole_5.3mm_M5_DIN965, F.Cu at (55.8, 82.8)
- added REF**: VIA-0.6mm, FDD_footprint:VIA-0.6mm, F.Cu at (80.0, 30.5)
- added REF**: VIA-0.6mm, FDD_footprint:VIA-0.6mm, F.Cu at (83.0, 29.5)
- added REF**: VIA-0.6mm, FDD_footprint:VIA-0.6mm, F.Cu at (81.0, 29.5)
- added REF**: VIA-0.6mm, FDD_footprint:VIA-0.6mm, F.Cu at (84.0, 28.5)
- added REF**: VIA-0.6mm, FDD_footprint:VIA-0.6mm, F.Cu at (82.0, 28.5)
- added REF**: VIA-0.6mm, FDD_footprint:VIA-0.6mm, F.Cu at (80.0, 28.5)
- added REF**: VIA-0.6mm, FDD_footprint:VIA-0.6mm, F.Cu at (83.0, 27.5)
- R1, R2, R3, R4, R5, R6, R7: footprint Resistors_THT:R_Axial_DIN0204_L3.6mm_D1.6mm_P5.08mm_Horizontal -> Resistors_THT:R_Axial_DIN0204_L3.6mm_D1.6mm_P2.54mm_Vertical
- U1, U10, U11, U12, U13, U14, U15, U16, U17, U18, U19, U2, U21, U22, U23, U24, U25, U26, U3, U4, U5, U6, U7, U8, U9: footprint Housings_DIP:DIP-16_W7.62mm_Socket_LongPads -> Housings_DIP:DIP-16_W7.62mm_Socket
- U20: footprint FDD_footprint:ESP8266_D1_Mini -> FDD_footprint:ESP8266_D1_Mini_cropped
- U27: footprint TO_SOT_Packages_THT:TO-220_Horizontal -> TO_SOT_Packages_THT:TO-220_Vertical
- U28: footprint Housings_DIP:DIP-28_W7.62mm_Socket_LongPads -> Housings_DIP:DIP-28_W7.62mm_Socket
- moved C5 177.2 mm to (80.0, 43.2), turned to 180 degrees
- moved R4 165.7 mm to (112.8, 26.9)
- moved R7 165.4 mm to (87.9, 32.5), turned to 90 degrees
- moved C7 163.8 mm to (93.0, 26.9), turned to 180 degrees
- moved C3 156.0 mm to (62.5, 37.8), turned to 270 degrees
- moved R1 150.8 mm to (120.9, 43.2), turned to 90 degrees
- moved R3 150.0 mm to (119.9, 26.9), turned to 180 degrees
- moved C4 149.7 mm to (72.6, 39.9), turned to 90 degrees
- moved R2 145.1 mm to (118.4, 40.6), turned to 270 degrees
- moved R6 144.0 mm to (118.4, 38.1), turned to 90 degrees
- moved U28 141.6 mm to (115.8, 35.6), turned to 270 degrees
- moved Y1 140.8 mm to (99.1, 31.2), turned to 180 degrees
- moved C8 126.6 mm to (79.2, 39.1), turned to 90 degrees
- moved P4 125.1 mm to (111.8, 49.8), turned to 90 degrees
- moved C6 121.2 mm to (96.8, 26.9)
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Connections:
- U20 pad 10: Net-(D1-Pad2) -> GND
- U20 pad 11: Net-(D2-Pad2) -> Net-(U20-Pad11)
- U20 pad 12: Net-(D3-Pad2) -> Net-(D1-Pad2)
- U20 pad 13: Net-(U20-Pad13) -> Net-(D2-Pad2)
- U20 pad 14: Net-(U20-Pad14) -> Net-(D3-Pad2)
- U20 pad 15: Net-(U20-Pad15) -> Net-(R1-Pad1)
- U20 pad 16: Net-(U20-Pad16) -> /Driver/ATM_RX
- U20 pad 9: Net-(U20-Pad9) -> +5V
Routing:
- net +5V: track 0.00 -> 701.8 mm, vias 0 -> 36
- net +12V: track 0.00 -> 648.8 mm, vias 0 -> 26
- net /DATA_X: track 0.00 -> 362.7 mm, vias 0 -> 7
- net /DATA_Y: track 0.00 -> 269.7 mm, vias 0 -> 11
- net /OE: track 0.00 -> 227.5 mm, vias 0 -> 17
- net /X_S_Latch: track 0.00 -> 109.7 mm, vias 0 -> 10
- net GND: track 0.00 -> 109.4 mm, vias 0 -> 7
- net /Y_S_Clock: track 0.00 -> 106.7 mm, vias 0 -> 9
- net /X_S_Clock: track 0.00 -> 105.5 mm, vias 0 -> 5
- net /Y_S_Latch: track 0.00 -> 101.3 mm, vias 0 -> 5
- net /EN_X1: track 122.3 -> 23.0 mm, vias 0 -> 2
- net /-Y16: track 110.3 -> 19.8 mm, vias 0 -> 2
- net /X12: track 136.7 -> 53.0 mm, vias 0 -> 2
- net /-Y15: track 101.7 -> 19.2 mm, vias 0 -> 3
- net /X10: track 119.9 -> 40.0 mm, vias 0 -> 2
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- added copper zone on B.Cu, net GND
- added copper zone on F.Cu, net GND
Other:
- board outline added: 100 x 100 mm
- board text added: "Pakue (2018)"
- board text added: "X2"
- board text added: "X24"
- board text added: "Y1+"
- board text added: "Y1-"
- board text added: "Y16-"
- board text added: "Y8+"
- board text added: "Y8-"
- board text added: "Y9+"

Commit message: PCB v1.1, minor fixes in connector and silkscreen layout
Parts:
- P1: footprint Pin_Headers:Pin_Header_Straight_2x13_Pitch2.54mm -> Pin_Headers:Pin_Header_Straight_2x12_Pitch2.54mm

Commit message: removed old ESP code
Parts:
- P1: footprint Pin_Headers:Pin_Header_Straight_2x12_Pitch2.54mm -> Pin_Headers:Pin_Header_Straight_2x13_Pitch2.54mm
